File: minitoy.kicad_pcb (KiCad board)
At the start: 2 copper layers, 0 parts

Commit message: Start layout
Parts:
- added C1: 0.01uF, Capacitors_SMD:C_0603, F.Cu at (111.6, 127.3)
- added C10: 0.01uF, Capacitors_SMD:C_0603, F.Cu at (126.6, 132.0)
- added C11: 0.1uF, Capacitors_SMD:C_0603, F.Cu at (129.3, 132.1)
- added C12: 0.01uF, Capacitors_SMD:C_0603, F.Cu at (123.9, 135.5)
- added C13: 0.01uF, Capacitors_SMD:C_0603, F.Cu at (120.4, 138.2)
- added C14: 0.1uF, Capacitors_SMD:C_0603, F.Cu at (222.8, 34.9)
- added C15: 0.1uF, Capacitors_SMD:C_0603, F.Cu at (227.6, 30.0)
- added C16: 1.0uF, Capacitors_SMD:C_0603, F.Cu at (212.1, 46.0)
- added C17: 1.0uF, Capacitors_SMD:C_0603, F.Cu at (229.9, 24.8)
- added C18: 47uF, Capacitors_SMD:CP_Elec_5x5.3, F.Cu at (175.5, 47.5)
- added C19: 1.0uF, Capacitors_SMD:C_0603, F.Cu at (207.3, 46.0)
- added C2: 0.1uF, Capacitors_SMD:C_0603, F.Cu at (227.6, 34.9)
- added C20: 1.0uF, Capacitors_SMD:C_0603, F.Cu at (218.3, 40.8)
- added C21: 47uF, Capacitors_SMD:CP_Elec_5x5.3, F.Cu at (185.5, 36.6)
- added C22: 1.0uF, Capacitors_SMD:C_0603, F.Cu at (222.8, 30.0)
- added C23: 1.0uF, Capacitors_SMD:C_0603, F.Cu at (213.5, 40.8)
- added C24: 47uF, Capacitors_SMD:CP_Elec_5x5.3, F.Cu at (224.3, 120.5)
- added C3: 0.01uF, Capacitors_SMD:C_0603, F.Cu at (124.4, 128.2)
- added C4: 0.01uF, Capacitors_SMD:C_0603, F.Cu at (108.1, 131.0)
- added C5: 0.1uF, Capacitors_SMD:C_0603, F.Cu at (105.3, 131.0)
- added C6: 1uF, Capacitors_SMD:C_0603, F.Cu at (102.7, 131.0)
- added C7: 0.01uF, Capacitors_SMD:C_0603, F.Cu at (126.6, 128.2)
- added C8: 0.1uF, Capacitors_SMD:C_0603, F.Cu at (128.3, 128.2)
- added C9: 1uF, Capacitors_SMD:C_0603, F.Cu at (130.1, 128.2)
- added D1: LED_ARGB, LEDs:LED_Cree-PLCC4_3.2x2.8mm_CCW, F.Cu at (128.8, 109.5)
- added D10: D_Schottky, Diodes_SMD:D_SOD-123, F.Cu at (177.7, 65.0)
- added D2: LED, LEDs:LED_0603, F.Cu at (123.1, 112.2)
- added D3: LED, LEDs:LED_0603, F.Cu at (121.1, 111.9)
- added D4: LED, LEDs:LED_0603, F.Cu at (119.4, 112.0)
- added D5: LED, LEDs:LED_0603, F.Cu at (116.5, 111.8)
- added D6: LED, LEDs:LED_0603, F.Cu at (114.6, 112.4)
- added D7: LED, LEDs:LED_0603, F.Cu at (112.9, 113.0)
- added D8: LED, LEDs:LED_0603, F.Cu at (109.7, 112.9)
- added D9: LED, LEDs:LED_0603, F.Cu at (107.1, 112.6)
- added J1: Conn_01x06, Pin_Headers:Pin_Header_Straight_1x06_Pitch2.54mm, F.Cu at (113.5, 60.5)
- added J2: PMOD1, Socket_Strips:Socket_Strip_Angled_2x06_Pitch2.54mm, F.Cu at (92.5, 64.1)
- added J3: PMOD2, Socket_Strips:Socket_Strip_Angled_2x06_Pitch2.54mm, F.Cu at (97.8, 31.9)
- added J4: USB_B_Micro, Connectors:USB_Micro-B_10103594-0001LF, F.Cu at (80.0, 142.6)
- added R1: 270, Resistors_SMD:R_0603, F.Cu at (122.9, 107.1)
- added R10: 10k, Resistors_SMD:R_0603, F.Cu at (208.9, 35.9)
- added R11: 100, Resistors_SMD:R_0603, F.Cu at (213.7, 30.7)
- added R12: 100, Resistors_SMD:R_0603, F.Cu at (225.3, 19.9)
- added R13: 100, Resistors_SMD:R_0603, F.Cu at (198.2, 45.6)
- added R14: 100, Resistors_SMD:R_0603, F.Cu at (220.8, 24.8)
- added R15: 100, Resistors_SMD:R_0603, F.Cu at (232.0, 14.7)
- added R16: 100, Resistors_SMD:R_0603, F.Cu at (204.4, 40.5)
- added R17: 100, Resistors_SMD:R_0603, F.Cu at (208.9, 41.0)
- added R18: 100, Resistors_SMD:R_0603, F.Cu at (181.9, 49.0)
- added R19: 10k, Resistors_SMD:R_0603, F.Cu at (213.4, 35.9)
- added R2: 270, Resistors_SMD:R_0603, F.Cu at (121.1, 107.0)
- added R20: 10k, Resistors_SMD:R_0603, F.Cu at (200.0, 35.3)
- added R21: 10k, Resistors_SMD:R_0603, F.Cu at (216.4, 20.4)
- added R22: 10k, Resistors_SMD:R_0603, F.Cu at (211.9, 25.6)
- added R23: 10k, Resistors_SMD:R_0603, F.Cu at (193.7, 41.6)
- added R24: 10k, Resistors_SMD:R_0603, F.Cu at (186.4, 49.3)
- added R3: 270, Resistors_SMD:R_0603, F.Cu at (119.2, 107.1)
- added R4: 270, Resistors_SMD:R_0603, F.Cu at (116.8, 107.0)
- added R5: 270, Resistors_SMD:R_0603, F.Cu at (114.4, 107.7)
- added R6: 270, Resistors_SMD:R_0603, F.Cu at (112.6, 107.8)
- added R7: 270, Resistors_SMD:R_0603, F.Cu at (109.5, 107.6)
- added R8: 270, Resistors_SMD:R_0603, F.Cu at (106.9, 107.3)
- added R9: 10k, Resistors_SMD:R_0603, F.Cu at (209.2, 30.7)
- added SW1: SW_Push, Buttons_Switches_THT:SW_PUSH_6mm, F.Cu at (196.8, 10.1)
- added SW2: SW_Push, Buttons_Switches_THT:SW_PUSH_6mm, F.Cu at (173.0, 34.7)
- added SW3: SW_Push, Buttons_Switches_THT:SW_PUSH_6mm, F.Cu at (206.9, 10.1)
- added SW4: SW_Push, Buttons_Switches_THT:SW_PUSH_6mm, F.Cu at (193.0, 21.8)
- added U1: ICE40UP5K-SG48, Housings_DFN_QFN:QFN-48-1EP_7x7mm_Pitch0.5mm, F.Cu at (117.7, 131.9)
- added U2: ESP-12E, RF_Modules:ESP-12E, F.Cu at (240.6, 45.0)
- added U3: MIC5504-1.2YM5, TO_SOT_Packages_SMD:SOT-23-5_HandSoldering, F.Cu at (143.8, 129.2)
- added U4: MIC5504-3.3YM5, TO_SOT_Packages_SMD:SOT-23-5_HandSoldering, F.Cu at (143.6, 123.0)
- added U5: MIC5504-3.3YM5, TO_SOT_Packages_SMD:SOT-23-5_HandSoldering, F.Cu at (143.7, 135.4)
Other:
- copper layers 2 -> 4
