File: minitoy.sch (KiCad schematic (older format))
At the start: 35 parts

Commit message: Change ESP reset scheme and UART connection
Parts:
- removed R?: 10k, symbol Device:R_Small
- added C?: 0.1uF, Capacitors_SMD:C_0603_HandSoldering, symbol Device:C_Small
- added D?: D_Schottky, symbol Device:D_Schottky
- added D?: LED_RGB, symbol Device:LED_RGB
- added J?: Conn_01x06, symbol Connector_Generic:Conn_01x06
Connections:
- net labels added: ESP_PROG
- net labels removed: ESP_RESET, UART_BOOT_EN
- wire segments 126 -> 140
- no-connect marks 9 -> 11
Other:
- note added: "3.3V"
- note added: "CTS"
- note added: "DTR"
- note added: "FTDI 3.3V UART"
- note added: "GND"
- note added: "RXD"
- note added: "TXD"

Commit message: Rough schematic complete.
Parts:
- added C? (x2): 0.1uF, Capacitors_SMD:C_0603_HandSoldering, symbol Device:C_Small
- added D? (x8): LED, symbol Device:LED
- added J?: PMOD1, symbol Connector_Generic:Conn_02x06_Top_Bottom
- added J?: PMOD2, symbol Connector_Generic:Conn_02x06_Top_Bottom
- added J?: USB_B_Micro, symbol Connector_Specialized:USB_B_Micro
- added R? (x8): 270, symbol Device:R_Small
- added R?: 100, symbol Device:R_Small
- added R? (x4): 10k, symbol Device:R_Small
- added SW? (x4): SW_Push, symbol Switch:SW_Push
Connections:
- net labels added: BTN0, BTN1, BTN2, BTN3, FPGA_INT, FPGA_LED_0, FPGA_LED_1, FPGA_LED_2, FPGA_LED_3, FPGA_LED_4, FPGA_LED_5, FPGA_LED_6, FPGA_LED_7, PMOD-1.1, PMOD-1.10, PMOD-1.2, PMOD-1.3, PMOD-1.4, PMOD-1.7, PMOD-1.8, PMOD-1.9, PMOD-2.1, PMOD-2.10, PMOD-2.2, PMOD-2.3, PMOD-2.4, PMOD-2.7, PMOD-2.8, PMOD-2.9
- wire segments 140 -> 274
- no-connect marks 11 -> 14

Commit message: Start layout
Parts:
- removed D?: LED_RGB, symbol Device:LED_RGB
- added C18, C21, C24: 47uF, Capacitors_SMD:CP_Elec_5x5.3, symbol Device:CP_Small
- added D1: LED_ARGB, LEDs:LED_Cree-PLCC4_3.2x2.8mm_CCW, symbol Device:LED_ARGB
- D10: renamed from D?; footprint (none) -> Diodes_SMD:D_SOD-123
- D2, D3, D4, D5, D6, D7, D8, D9: renamed from D?; footprint (none) -> LEDs:LED_0603_HandSoldering
- J1: renamed from J?; footprint (none) -> Pin_Headers:Pin_Header_Straight_1x06_Pitch2.54mm
- J2, J3: renamed from J?; footprint (none) -> Socket_Strips:Socket_Strip_Angled_2x06_Pitch2.54mm
- J4: renamed from J?; footprint (none) -> Connectors:USB_Micro-B_10103594-0001LF
- R1, R10, R11, R12, R13, R15, R16, R17, R18, R19, R2, R20, R21, R22, R23, R24, R3, R4, R5, R6, R7, R8, R9: renamed from R?; footprint (none) -> Resistors_SMD:R_0603_HandSoldering
- SW1, SW2, SW3, SW4: renamed from SW?; footprint (none) -> Buttons_Switches_THT:SW_PUSH_6mm
- U1: renamed from U?; footprint (none) -> Housings_DFN_QFN:QFN-48-1EP_7x7mm_Pitch0.5mm
- U2: renamed from U?; footprint RF_Module:ESP-12E -> RF_Modules:ESP-12E
- U3, U4, U5: renamed from U?; footprint Package_TO_SOT_SMD:SOT-23-5 -> TO_SOT_Packages_SMD:SOT-23-5_HandSoldering
- gave numbers to parts that had none: 22
Connections:
- wire segments 274 -> 281

Commit message: Remove blinkenlights and buttons, add another PMOD socket
Parts:
- removed D2, D3, D4, D5, D6, D7, D8, D9: LED, LEDs:LED_0603_HandSoldering, symbol Device:LED
- removed R1, R2, R3, R4, R5, R6, R7, R8: 270, Resistors_SMD:R_0603_HandSoldering, symbol Device:R_Small
- removed R21, R22, R23, R24: 10k, Resistors_SMD:R_0603_HandSoldering, symbol Device:R_Small
- removed SW1, SW2, SW3, SW4: SW_Push, Buttons_Switches_THT:SW_PUSH_6mm, symbol Switch:SW_Push
- added C25: 0.1uF, Capacitors_SMD:C_0603_HandSoldering, symbol Device:C_Small
- added J5: PMOD3, Socket_Strips:Socket_Strip_Angled_2x06_Pitch2.54mm, symbol Connector_Generic:Conn_02x06_Top_Bottom
Connections:
- net labels added: PMOD-3.1, PMOD-3.10, PMOD-3.2, PMOD-3.3, PMOD-3.4, PMOD-3.7, PMOD-3.8, PMOD-3.9
- net labels removed: BTN0, BTN1, BTN2, BTN3, FPGA_LED_0, FPGA_LED_1, FPGA_LED_2, FPGA_LED_3, FPGA_LED_4, FPGA_LED_5, FPGA_LED_6, FPGA_LED_7
- wire segments 281 -> 250
- no-connect marks 14 -> 18

Commit message: More consolidation of the board
Parts:
- removed J2: PMOD1, Socket_Strips:Socket_Strip_Angled_2x06_Pitch2.54mm, symbol Connector_Generic:Conn_02x06_Top_Bottom
- removed J3: PMOD2, Socket_Strips:Socket_Strip_Angled_2x06_Pitch2.54mm, symbol Connector_Generic:Conn_02x06_Top_Bottom
- removed J5: PMOD3, Socket_Strips:Socket_Strip_Angled_2x06_Pitch2.54mm, symbol Connector_Generic:Conn_02x06_Top_Bottom
- added J2: PMOD1, Socket_Strips:Socket_Strip_Angled_2x06_Pitch2.54mm, symbol Connector_Generic:Conn_02x06_Odd_Even
- added J3: PMOD2, Socket_Strips:Socket_Strip_Angled_2x06_Pitch2.54mm, symbol Connector_Generic:Conn_02x06_Odd_Even
- added J5: PMOD3, Socket_Strips:Socket_Strip_Angled_2x06_Pitch2.54mm, symbol Connector_Generic:Conn_02x06_Odd_Even
Changed lines of the file:
@@
 	1    0    0    -1
 $EndComp
-Text GLabel 1950 2100 0    39   Output ~ 0
+Text GLabel 1950 2100 0    39   BiDi ~ 0
+PMOD-3.8
+Text GLabel 1950 2200 0    39   BiDi ~ 0
+PMOD-3.9
+Text GLabel 1950 2300 0    39   BiDi ~ 0
+PMOD-3.10
+Text GLabel 3000 1400 1    39   BiDi ~ 0
+PMOD-3.1
+Text GLabel 2900 1400 1    39   BiDi ~ 0
+PMOD-3.2
+Text GLabel 2800 1400 1    39   BiDi ~ 0
 PMOD-3.3
-Text GLabel 1950 2200 0    39   Output ~ 0
-PMOD-3.2
-Text GLabel 1950 2300 0    39   Output ~ 0
-PMOD-3.1
-Text GLabel 3000 1400 1    39   Output ~ 0
-PMOD-3.10
-Text GLabel 2900 1400 1    39   Output ~ 0
-PMOD-3.9
-Text GLabel 2800 1400 1    39   Output ~ 0
-PMOD-3.8
-Text GLabel 2700 1400 1    39   Output ~ 0
+Text GLabel 2700 1400 1    39   BiDi ~ 0
+PMOD-3.4
+Text GLabel 2600 1400 1    39   BiDi ~ 0
 PMOD-3.7
-Text GLabel 2600 1400 1    39   Output ~ 0
-PMOD-3.4
 Wire Wire Line
 	1950 2100 2050 2100
@@
 Wire Wire Line
 	3000 1400 3000 1450
-$Comp
-L Connector_Generic:Conn_02x06_Top_Bottom J2
-U 1 1 5A985BCC
-P 4950 4900
-F 0 "J2" H 5000 5317 50  0000 C CNN
-F 1 "PMOD1" H 5000 5226 50  0000 C CNN
-F 2 "Socket_Strips:Socket_Strip_Angled_2x06_Pitch2.54mm" H 4950 4900 50  0001 C CNN
-F 3 "~" H 4950 4900 50  0001 C CNN
-	1    4950 4900
-	1    0    0    -1
-$EndComp
 Wire Wire Line
 	4750 5100 4600 5100
@@
 Wire Wire Line
 	3200 3750 3200 3650
-$Comp
-L Connector_Generic:Conn_02x06_Top_Bottom J3
-U 1 1 5AA5BE7F
-P 6550 4900
-F 0 "J3" H 6600 5317 50  0000 C CNN
-F 1 "PMOD2" H 6600 5226 50  0000 C CNN
-F 2 "Socket_Strips:Socket_Strip_Angled_2x06_Pitch2.54mm" H 6550 4900 50  0001 C CNN
-F 3 "~" H 6550 4900 50  0001 C CNN
-	1    6550 4900
-	1    0    0    -1
-$EndComp
 Wire Wire Line
 	6350 5100 6200 5100
@@
 	0    -1   -1   0
 $EndComp
-$Comp
-L Connector_Generic:Conn_02x06_Top_Bottom J5
-U 1 1 5A90DDFA
-P 8150 4900
-F 0 "J5" H 8200 5317 50  0000 C CNN
-F 1 "PMOD3" H 8200 5226 50  0000 C CNN
-F 2 "Socket_Strips:Socket_Strip_Angled_2x06_Pitch2.54mm" H 8150 4900 50  0001 C CNN
-F 3 "~" H 8150 4900 50  0001 C CNN
-	1    8150 4900
-	1    0    0    -1
-$EndComp
 Wire Wire Line
 	7950 5100 7800 5100
@@
 NoConn ~ 3200 1450
 NoConn ~ 3600 1450
+$Comp
+L Connector_Generic:Conn_02x06_Odd_Even J2
+U 1 1 5A98A244
+P 4950 4900
+F 0 "J2" H 5000 5317 50  0000 C CNN
+F 1 "PMOD1" H 5000 5226 50  0000 C CNN
+F 2 "Socket_Strips:Socket_Strip_Angled_2x06_Pitch2.54mm" H 4950 4900 50  0001 C CNN
+F 3 "~" H 4950 4900 50  0001 C CNN
+	1    4950 4900
+	1    0    0    -1
+$EndComp
+$Comp
+L Connector_Generic:Conn_02x06_Odd_Even J3
+U 1 1 5A98A3A3
+P 6550 4900
+F 0 "J3" H 6600 5317 50  0000 C CNN
+F 1 "PMOD2" H 6600 5226 50  0000 C CNN
+F 2 "Socket_Strips:Socket_Strip_Angled_2x06_Pitch2.54mm" H 6550 4900 50  0001 C CNN
+F 3 "~" H 6550 4900 50  0001 C CNN
+	1    6550 4900
+	1    0    0    -1
+$EndComp
+$Comp
+L Connector_Generic:Conn_02x06_Odd_Even J5
+U 1 1 5A98A433
+P 8150 4900
+F 0 "J5" H 8200 5317 50  0000 C CNN
+F 1 "PMOD3" H 8200 5226 50  0000 C CNN
+F 2 "Socket_Strips:Socket_Strip_Angled_2x06_Pitch2.54mm" H 8150 4900 50  0001 C CNN
+F 3 "~" H 8150 4900 50  0001 C CNN
+	1    8150 4900
+	1    0    0    -1
+$EndComp
 $EndSCHEMATC

Commit message: More layout changes, remove a PMOD socket for easier routing
Parts:
- removed C15: 0.1uF, Capacitors_SMD:C_0603_HandSoldering, symbol Device:C_Small
- removed J3: PMOD2, Socket_Strips:Socket_Strip_Angled_2x06_Pitch2.54mm, symbol Connector_Generic:Conn_02x06_Odd_Even
- J5: value PMOD3 -> PMOD2
Connections:
- net labels added: VCCPLL
- net labels removed: PMOD-3.1, PMOD-3.10, PMOD-3.2, PMOD-3.3, PMOD-3.4, PMOD-3.7, PMOD-3.8, PMOD-3.9
- wire segments 250 -> 221
- no-connect marks 18 -> 26

Commit message: Routing done, but cleanup needed
Parts:
- removed C7: 0.01uF, Capacitors_SMD:C_0603_HandSoldering, symbol Device:C_Small
- removed C8: 0.1uF, Capacitors_SMD:C_0603_HandSoldering, symbol Device:C_Small
- removed C9: 1uF, Capacitors_SMD:C_0603_HandSoldering, symbol Device:C_Small
- removed R11, R12, R13, R15, R16, R17, R18: 100, Resistors_SMD:R_0603_HandSoldering, symbol Device:R_Small
- C1, C13, C3: value 0.01uF -> 0.1uF
- renumbered C19 to C16, C20 to C17, C21 to C18, C16 to C19, C17 to C20, C18 to C21, U4 to U3, U3 to U4
Connections:
- net labels removed: FPGA_PWR_EN
- wire segments 221 -> 213
- no-connect marks 26 -> 20

Commit message: v0.2: fix ESP POR straps and reset, fix typo on serial connector
Parts:
- added R1: 10k, Resistors_SMD:R_0603_HandSoldering, symbol Device:R_Small
- C2: value 0.1uF -> 1uF
Connections:
- no-connect marks 20 -> 19
Other:
- note added: "5V"
- note removed: "3.3V"
- note removed: "Master boot mode"
Changed lines of the file:
@@
 Wire Wire Line
 	8650 3700 8650 3750
-Text Notes 8900 3650 0    39   ~ 0
-Master boot mode
 $Comp
 L Device:R_Small R19
 U 1 1 5A874DC0
-P 8400 3600
-F 0 "R19" H 8341 3554 50  0000 R CNN
-F 1 "10k" H 8341 3645 50  0000 R CNN
-F 2 "Resistors_SMD:R_0603_HandSoldering" H 8400 3600 50  0001 C CNN
-F 3 "~" H 8400 3600 50  0001 C CNN
-	1    8400 3600
+P 8650 2550
+F 0 "R19" H 8591 2504 50  0000 R CNN
+F 1 "10k" H 8591 2595 50  0000 R CNN
+F 2 "Resistors_SMD:R_0603_HandSoldering" H 8650 2550 50  0001 C CNN
+F 3 "~" H 8650 2550 50  0001 C CNN
+	1    8650 2550
 	-1   0    0    1
 $EndComp
-Wire Wire Line
-	8300 2700 8400 2700
-Wire Wire Line
-	8400 2700 8400 3500
-Wire Wire Line
-	8400 3700 8400 3750
-Wire Wire Line
-	8400 3750 8550 3750
 $Comp
 L power:GND #PWR021
 U 1 1 5A876272
-P 8550 3750
-F 0 "#PWR021" H 8550 3500 50  0001 C CNN
-F 1 "GND" H 8555 3577 50  0000 C CNN
-F 2 "" H 8550 3750 50  0001 C CNN
-F 3 "" H 8550 3750 50  0001 C CNN
-	1    8550 3750
-	1    0    0    -1
-$EndComp
-Connection ~ 8550 3750
-Wire Wire Line
-	8550 3750 8650 3750
-Wire Notes Line
-	8300 3500 9450 3500
-Wire Notes Line
-	9450 3500 9450 3700
-Wire Notes Line
-	9450 3700 8300 3700
-Wire Notes Line
-	8300 3700 8300 3500
+P 8650 3750
+F 0 "#PWR021" H 8650 3500 50  0001 C CNN
+F 1 "GND" H 8655 3577 50  0000 C CNN
+F 2 "" H 8650 3750 50  0001 C CNN
+F 3 "" H 8650 3750 50  0001 C CNN
+	1    8650 3750
+	1    0    0    -1
+$EndComp
 $Comp
 L Device:R_Small R10
@@
 Wire Wire Line
 	8300 2200 9050 2200
-Text GLabel 6100 2100 0    39   Input ~ 0
+Text GLabel 6000 2000 0    39   Input ~ 0
 ESP_PROG
 Wire Wire Line
-	6450 1850 6450 2100
+	6450 1850 6450 2000
 NoConn ~ 8300 2500
 Text GLabel 2800 3750 3    39   Input ~ 0
@@
 Text Notes 3600 3750 1    50   ~ 0
 I3C
-NoConn ~ 6500 2000
 Wire Wire Line
 	7400 3900 7400 4000
@@
 L Device:C_Small C2
 U 1 1 5A88AFAF
-P 6250 2100
-F 0 "C2" V 6300 1950 50  0000 L CNN
-F 1 "0.1uF" V 6350 1950 50  0000 L CNN
-F 2 "Capacitors_SMD:C_0603_HandSoldering" H 6250 2100 50  0001 C CNN
-F 3 "~" H 6250 2100 50  0001 C CNN
-	1    6250 2100
+P 6150 2000
+F 0 "C2" V 6200 1850 50  0000 L CNN
+F 1 "1uF" V 6250 1850 50  0000 L CNN
+F 2 "Capacitors_SMD:C_0603_HandSoldering" H 6150 2000 50  0001 C CNN
+F 3 "~" H 6150 2000 50  0001 C CNN
+	1    6150 2000
 	0    1    1    0
 $EndComp
 Wire Wire Line
-	6100 2100 6150 2100
-Wire Wire Line
-	6350 2100 6450 2100
+	6000 2000 6050 2000
 $Comp
 L Device:D_Schottky D10
@@
 Text Notes 9800 4550 0    50   ~ 0
 FTDI 3.3V UART
-Wire Wire Line
-	6450 2100 6450 2200
-Wire Wire Line
-	6450 2200 6500 2200
-Connection ~ 6450 2100
 Text Notes 9600 3900 0    39   ~ 0
 DTR
@@
 GND
 Text Notes 9600 4200 0    39   ~ 0
-3.3V
+5V
 Text Notes 9600 4300 0    39   ~ 0
 CTS
@@
 	8950 2000 9050 2000
 Wire Wire Line
-	9050 2700 8400 2700
-Connection ~ 8400 2700
-Wire Wire Line
 	9050 2900 8300 2900
 Wire Wire Line
@@
 	5150 2700 4250 2700
 $Comp
-L power:GND #PWR?
+L power:GND #PWR0101
 U 1 1 5A9D7127
 P 4950 2900
-F 0 "#PWR?" H 4950 2650 50  0001 C CNN
+F 0 "#PWR0101" H 4950 2650 50  0001 C CNN
 F 1 "GND" H 4955 2727 50  0000 C CNN
 F 2 "" H 4950 2900 50  0001 C CNN
@@
 Wire Wire Line
 	4950 2800 4950 2900
+Wire Wire Line
+	6250 2000 6450 2000
+$Comp
+L Device:R_Small R1
+U 1 1 5AA8ED30
+P 6300 1750
+F 0 "R1" H 6450 1700 50  0000 R CNN
+F 1 "10k" H 6500 1800 50  0000 R CNN
+F 2 "Resistors_SMD:R_0603_HandSoldering" H 6300 1750 50  0001 C CNN
+F 3 "~" H 6300 1750 50  0001 C CNN
+	1    6300 1750
+	-1   0    0    1
+$EndComp
+Wire Wire Line
+	6300 1650 6300 1600
+Wire Wire Line
+	6300 1600 6450 1600
+Connection ~ 6450 1600
+Wire Wire Line
+	6300 1850 6300 2200
+Wire Wire Line
+	6300 2200 6500 2200
+Wire Wire Line
+	6450 2000 6500 2000
+Connection ~ 6450 2000
+$Comp
+L power:+3.3VA #PWR0102
+U 1 1 5AAC04AE
+P 8650 2450
+F 0 "#PWR0102" H 8650 2300 50  0001 C CNN
+F 1 "+3.3VA" H 8650 2600 50  0000 C CNN
+F 2 "" H 8650 2450 50  0001 C CNN
+F 3 "" H 8650 2450 50  0001 C CNN
+	1    8650 2450
+	1    0    0    -1
+$EndComp
+Wire Wire Line
+	8300 2700 8650 2700
+Wire Wire Line
+	8650 2650 8650 2700
+Connection ~ 8650 2700
+Wire Wire Line
+	8650 2700 9050 2700
 $EndSCHEMATC
